File: floppy_bracket/floppy_bracket.kicad_sch (KiCad schematic)
At the start: 16 parts

Commit message: Finalize bracket
Parts:
- H13, H14, H15, H16: footprint MountingHole:MountingHole_3.2mm_M3_Pad -> MountingHole:MountingHole_3.2mm_M3
Changed lines of the file:
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@@
       (effects (font (size 1.27 1.27)) (justify left))
     )
-    (property "Footprint" "MountingHole:MountingHole_3.2mm_M3_Pad" (id 2) (at 123.19 125.73 0)
+    (property "Footprint" "MountingHole:MountingHole_3.2mm_M3" (id 2) (at 123.19 125.73 0)
       (effects (font (size 1.27 1.27)) hide)
     )
@@
       (effects (font (size 1.27 1.27)) (justify left))
     )
-    (property "Footprint" "MountingHole:MountingHole_3.2mm_M3_Pad" (id 2) (at 123.19 132.08 0)
+    (property "Footprint" "MountingHole:MountingHole_3.2mm_M3" (id 2) (at 123.19 132.08 0)
       (effects (font (size 1.27 1.27)) hide)
     )
@@
       (effects (font (size 1.27 1.27)) (justify left))
     )
-    (property "Footprint" "MountingHole:MountingHole_3.2mm_M3_Pad" (id 2) (at 123.19 138.43 0)
+    (property "Footprint" "MountingHole:MountingHole_3.2mm_M3" (id 2) (at 123.19 138.43 0)
       (effects (font (size 1.27 1.27)) hide)
     )
@@
       (effects (font (size 1.27 1.27)) (justify left))
     )
-    (property "Footprint" "MountingHole:MountingHole_3.2mm_M3_Pad" (id 2) (at 123.19 119.38 0)
+    (property "Footprint" "MountingHole:MountingHole_3.2mm_M3" (id 2) (at 123.19 119.38 0)
       (effects (font (size 1.27 1.27)) hide)
     )
@@
     )
     (path "/ed649220-2164-42c0-a046-6acec8dcb52a"
-      (reference "H13") (unit 1) (value "MountingHole") (footprint "MountingHole:MountingHole_3.2mm_M3_Pad")
+      (reference "H13") (unit 1) (value "MountingHole") (footprint "MountingHole:MountingHole_3.2mm_M3")
     )
     (path "/4b5f3762-af04-4ed2-8f07-a69a13d5c54d"
-      (reference "H14") (unit 1) (value "MountingHole") (footprint "MountingHole:MountingHole_3.2mm_M3_Pad")
+      (reference "H14") (unit 1) (value "MountingHole") (footprint "MountingHole:MountingHole_3.2mm_M3")
     )
     (path "/cb1dbec2-beda-4367-94c6-76c560f18bf1"
-      (reference "H15") (unit 1) (value "MountingHole") (footprint "MountingHole:MountingHole_3.2mm_M3_Pad")
+      (reference "H15") (unit 1) (value "MountingHole") (footprint "MountingHole:MountingHole_3.2mm_M3")
     )
     (path "/da60a574-7ec2-421a-ad07-3acb7e2edf90"
-      (reference "H16") (unit 1) (value "MountingHole") (footprint "MountingHole:MountingHole_3.2mm_M3_Pad")
-    )
-  )
+      (reference "H16") (unit 1) (value "MountingHole") (footprint "MountingHole:MountingHole_3.2mm_M3")
+    )
+  )
